File: display.kicad_sch (KiCad schematic)
At the start: 6 parts

Commit message: HW: PIO done
Other:
- title: (none) -> DL1414 display
Changed lines of the file:
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@@
 	(paper "A5")
 	(title_block
-		(date "2025-10-14")
+		(title "DL1414 display")
+		(date "2025-10-16")
 		(rev "A")
 		(company "A.K.")
