File: pocket80.kicad_pcb (KiCad board)
At the start: 4 copper layers, 68.6 x 107.3 mm, 137 parts, among them J1 USB_C_Receptacle_USB2.0_14P, J2 Conn_02x10_Odd_Even, J3 Conn_01x02, Q1 IRLML6402, Q2 BC847, SW1 F1, SW10 4, SW11 9, SW12 5, SW13 A, SW14 6, SW15 B, SW16 7, SW17 0, SW18 INC, SW19 1, SW2 F2, SW20 DEC, SW21 2, SW22 SEL, SW23 3, SW24 GO!, SW25 SW_Push_DPDT, SW26 RESET, SW3 F3, SW4 F4, SW5 C, SW6 D, SW7 E, SW8 F, SW9 8, U1 Z80CPU, U10 74HC00, U11 74HC138, U12 CH340N, U13 TP4056-42-ESOP8, U14 SX1308, U15 LM393, U16 74HC74, U17 28C256, U2 74HC244, U3 PIO-PLCC-44, U4 SIO3-PLCC-44, U5 CTC-PLCC-44, U6 NE555D, U7 74HC04, U8 62256, U9 24C512, Y1 3.6864M

Commit message: HW: Routing WIP
Parts:
- moved C6 0.13 mm to (145.4, 114.0)
Routing:
- net /CPU/~{RST}: track 0.00 -> 161.7 mm, vias 0 -> 8
- net /CPU/D3: track 76.7 -> 238.4 mm, vias 5 -> 10
- net /CPU/D6: track 33.6 -> 192.8 mm, vias 2 -> 9
- net /CPU/A0: track 73.6 -> 228.6 mm, vias 2 -> 9
- net /CPU/A1: track 69.4 -> 221.2 mm, vias 2 -> 11
- net /CPU/D1: track 77.8 -> 228.3 mm, vias 3 -> 10
- net /CPU/D2: track 89.0 -> 229.3 mm, vias 5 -> 10
- net /CPU/~{M1}: track 0.00 -> 137.7 mm, vias 0 -> 10
- net /CPU/D0: track 96.4 -> 234.1 mm, vias 2 -> 9
- net /CPU/~{SRST}: track 0.00 -> 136.4 mm, vias 0 -> 5
- net /CPU/~{RD}: track 0.00 -> 129.1 mm, vias 0 -> 9
- net /CPU/CLK: track 1.46 -> 118.5 mm, vias 1 -> 6
- net /CPU/~{DISP1}: track 0.00 -> 116.8 mm, vias 0 -> 2
- net /CPU/D4: track 73.3 -> 188.4 mm, vias 5 -> 14
- net /CPU/D5: track 64.9 -> 178.0 mm, vias 5 -> 8
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
Commit message: HW: Routing WIP
Parts:
- C31: moved to F.Cu
- U3: value PIO-PLCC-44 -> Z80 PIO
- U4: value SIO3-PLCC-44 -> Z80 SIO3
- U5: value CTC-PLCC-44 -> Z80 CTC
- moved R33 60.0 mm to (104.0, 96.8), turned to 180 degrees
- moved R34 59.8 mm to (104.0, 98.7), turned to 180 degrees
- moved C31 58.5 mm to (103.4, 94.4), turned to 180 degrees
- moved D12 48.8 mm to (103.3, 87.0), turned to 180 degrees
- moved U9 47.8 mm to (103.4, 91.9)
- moved D11 47.4 mm to (103.3, 84.7), turned to 180 degrees
- moved C11 2.17 mm to (157.1, 114.8), turned to 0 degrees
- moved C22 1.02 mm to (120.7, 84.6)
Routing:
- net /Expansion/PORTB0: track 0.00 -> 100.6 mm, vias 0 -> 3
- net /Expansion/PORTB1: track 0.00 -> 100.3 mm, vias 0 -> 1
- net /CTC/TO0: track 0.00 -> 100.1 mm, vias 0 -> 1
- net Net-(U3-PB2): track 0.00 -> 93.2 mm, vias 0 -> 15
- net Net-(U2-2A1): track 31.1 -> 110.4 mm, vias 4 -> 7
- net Net-(U2-2A0): track 39.6 -> 112.4 mm, vias 10 -> 13
- net Net-(U16B-C): track 6.81 -> 77.9 mm, vias 0 -> 1
- net /CTC/TO1: track 0.00 -> 44.6 mm, vias 0 -> 2
- net /PIO/IEI: track 0.00 -> 29.6 mm, vias 0 -> 2
- net GND: track 90.3 -> 112.8 mm, vias 51 -> 64
- net Net-(D11-K): track 0.00 -> 21.7 mm, vias 0 -> 4
- net /CTC/IEO: track 0.00 -> 19.1 mm, vias 0 -> 4
- net Net-(D11-A): track 7.86 -> 26.9 mm, vias 0 -> 2
- net Net-(D12-A): track 9.91 -> 23.8 mm, vias 0 -> 2
- net Net-(D12-K): track 0.00 -> 13.1 mm, vias 0 -> 4
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
Commit message: HW: Routing done
Routing:
- net Net-(D4-A): track 46.8 -> 72.9 mm, vias 0 -> 4
- net VCC: track 115.0 -> 119.8 mm, vias 43 -> 44
- net Net-(U6-TR): track 4.47 -> 7.54 mm, vias 0 -> 1
- net GND: track 112.8 -> 114.9 mm
- net Net-(U2-1A2): track 64.3 -> 66.3 mm
- net Net-(U15A-+): track 13.7 -> 15.8 mm
- net /CTC/TO0: track 100.1 -> 101.2 mm
- net /Expansion/PORTA6: vias 3 -> 2

Commit message: HW: Rev A
Parts:
- added REF**: OSHW-Logo2_7.3x6mm_SilkScreen, Symbol:OSHW-Logo2_7.3x6mm_SilkScreen, F.Cu at (160.5, 70.9)
- moved SW25 0.25 mm to (108.8, 39.9)
Routing:
- net Net-(Q1-G): track 3.30 -> 0.00 mm
- net Net-(C29-Pad2): track 5.78 -> 4.65 mm
- net GND: vias 64 -> 69
- added copper zone on F.Cu, net GND
Other:
- board text added: "A.K. 2025"
- board text added: "JLCJLCJLCJLC"
- board text added: "Pocket80"
- board text added: "Rev A"
